File: MySXRelay.kicad_pcb (KiCad board)
At the start: 4 copper layers, 36 x 36.6 mm, 65 parts, among them J1 AVR ISP, J2 PRG/BL0942, J3 Relay, Q1 2N7002, U2 BL0942, U3 BP2525X, U4 Si8642BB-B-IS1, U5 MCP1703Ax-180xxTT, U6 ATmega328PB-A, U7 AT25xxx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

Commit message: finish PCB afterr changing connector
Parts:
- R14, R15, R16, R17, R18: moved to B.Cu
- moved R16 27.5 mm to (169.7, 101.4)
- moved R15 27.2 mm to (165.1, 101.4)
- moved R17 25.2 mm to (170.8, 97.9), turned to -90 degrees
- moved R14 23.1 mm to (163.9, 97.9), turned to 90 degrees
- moved R18 20.5 mm to (170.2, 93.3), turned to -90 degrees
- moved C12 11.6 mm to (164.6, 94.1), turned to 90 degrees
- moved R13 8.91 mm to (163.1, 94.1), turned to 90 degrees
Routing:
- net N_IN: track 134.8 -> 162.1 mm, vias 29 -> 8
- net D2: track 45.0 -> 33.0 mm
- net Net-(U2-VP): track 18.6 -> 7.36 mm, vias 2 -> 1
- net L_IN: track 14.1 -> 23.9 mm
- net BL0942_TX: track 23.2 -> 18.1 mm
- net Net-(R16-Pad1): track 0.00 -> 2.19 mm
- net Net-(R14-Pad1): track 0.00 -> 2.15 mm
- net L_SENSE: track 0.00 -> 1.92 mm
- net Net-(R15-Pad1): track 0.00 -> 1.68 mm
- net BL0942_RX: track 42.4 -> 42.8 mm, vias 4 -> 3
Other:
- board text added: "MySXRelay v2.1"
- board text removed: "MySXRelay v2.0"

Commit message: change AP2204 to AP2202
Parts:
- U8: value AP2204K-ADJ -> AP2202K-5.0
Changed lines of the file:
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@@
 	(net 46 "/MCU/A1")
 	(net 47 "D8")
-	(net 48 "Net-(U8-ADJ)")
+	(net 48 "Net-(U8-BYP)")
 	(net 49 "D5")
 	(net 50 "D2")
@@
 			)
 		)
-		(property "Value" "AP2204K-ADJ"
+		(property "Value" "AP2202K-5.0"
 			(at 0 2.4 90)
 			(layer "F.Fab")
@@
 			)
 		)
-		(property "Datasheet" "https://www.diodes.com/assets/Datasheets/products_inactive_data/AP2204.pdf"
+		(property "Datasheet" "https://www.diodes.com/assets/Datasheets/AP2202.pdf"
 			(at 0 0 90)
 			(layer "F.Fab")
@@
 			(layers "F.Cu" "F.Paste" "F.Mask")
 			(roundrect_rratio 0.25)
-			(net 48 "Net-(U8-ADJ)")
-			(pinfunction "ADJ")
+			(net 48 "Net-(U8-BYP)")
+			(pinfunction "BYP")
 			(pintype "input")
 		)
@@
 			(layers "F.Cu" "F.Paste" "F.Mask")
 			(roundrect_rratio 0.25)
-			(net 48 "Net-(U8-ADJ)")
+			(net 48 "Net-(U8-BYP)")
 			(pintype "passive")
 		)
