File: mcu.kicad_sch (KiCad schematic)
At the start: 20 parts, among them J1 AVR ISP, Q1 2N7002, U6 ATmega328PB-A, U7 AT25xxx, X3 Switch/LED

Commit message: fix part names and datasheet links
Parts:
- U7: value AT25xxx -> AT25512
Changed lines of the file:
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@@
 	(label "RST"
 		(at 117.475 85.09 0)
-		(fields_autoplaced yes)
 		(effects
 			(font
@@
 	(label "LED"
 		(at 177.8 120.65 0)
-		(fields_autoplaced yes)
 		(effects
 			(font
@@
 	(label "SW"
 		(at 177.8 118.11 0)
-		(fields_autoplaced yes)
 		(effects
 			(font
@@
 	(label "A1"
 		(at 117.475 72.39 0)
-		(fields_autoplaced yes)
 		(effects
 			(font
@@
 			)
 		)
-		(property "Value" "AT25xxx"
+		(property "Value" "AT25512"
 			(at 196.5041 40.64 0)
 			(effects
@@
 			)
 		)
-		(property "Datasheet" "http://ww1.microchip.com/downloads/en/DeviceDoc/Atmel-8707-SEEPROM-AT25010B-020B-040B-Datasheet.pdf"
+		(property "Datasheet" "https://ww1.microchip.com/downloads/en/DeviceDoc/AT25512-SPI-Serial-EEPROM-512-Kbits-20006218A.pdf"
 			(at 194.31 48.26 0)
 			(effects

Commit message: replace RS485 low voltage side with single isolated transciever chip CA-IS3092W
Changed lines of the file:
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@@
 	(text "Switch"
 		(exclude_from_sim no)
-		(at 212.598 118.364 0)
+		(at 212.09 118.11 0)
 		(effects
 			(font
@@
 	(text "LED"
 		(exclude_from_sim no)
-		(at 197.358 147.574 0)
+		(at 196.85 147.32 0)
 		(effects
 			(font
@@
 	(text "MCU"
 		(exclude_from_sim no)
-		(at 93.091 133.35 0)
+		(at 92.71 133.35 0)
 		(effects
 			(font
@@
 	)
 	(label "RST"
-		(at 117.475 85.09 0)
+		(at 118.11 85.09 0)
 		(effects
 			(font
@@
 	)
 	(label "A1"
-		(at 117.475 72.39 0)
+		(at 118.11 72.39 0)
 		(effects
 			(font

Commit message: rework for proper clearence distances
Parts:
- R20, R22: value 1M -> 10k
Changed lines of the file:
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@@
 			)
 		)
-		(property "Value" "1M"
+		(property "Value" "10k"
 			(at 179.705 48.26 0)
 			(effects
@@
 			)
 		)
-		(property "Value" "1M"
+		(property "Value" "10k"
 			(at 133.985 80.01 0)
 			(effects
